File: EngineControl.kicad_pcb (KiCad board)
At the start: 0 parts

Commit message: Complete Rev0
Parts:
- added C1: 10uF, Capacitor_Tantalum_SMD:CP_EIA-3216-18_Kemet-A, F.Cu at (113.6, 126.6)
- added C10: 100nF, Capacitor_SMD:C_0402_1005Metric, F.Cu at (122.2, 105.1)
- added C11: 100uF, Capacitor_Tantalum_SMD:CP_EIA-7343-31_Kemet-D, F.Cu at (82.0, 99.7)
- added C12: 100u, Capacitor_Tantalum_SMD:CP_EIA-7343-31_Kemet-D, F.Cu at (82.0, 109.5)
- added C2: 100nF, Capacitor_SMD:C_0402_1005Metric, F.Cu at (107.4, 124.6)
- added C3: 1uF, Capacitor_Tantalum_SMD:CP_EIA-3216-18_Kemet-A, F.Cu at (94.2, 125.8)
- added C4: 100nF, Capacitor_SMD:C_0402_1005Metric, F.Cu at (111.4, 115.4)
- added C5: 100nF, Capacitor_SMD:C_0402_1005Metric, F.Cu at (97.4, 125.7)
- added C6: 100nF, Capacitor_SMD:C_0402_1005Metric, F.Cu at (102.4, 111.8)
- added C7: 100nF, Capacitor_SMD:C_0402_1005Metric, F.Cu at (100.0, 113.4)
- added C8: 10pF, Capacitor_SMD:C_0402_1005Metric, F.Cu at (94.4, 114.2)
- added C9: 10pF, Capacitor_SMD:C_0402_1005Metric, F.Cu at (94.4, 121.8)
- added D1: LED_HeartBeat, LED_SMD:LED_0603_1608Metric, F.Cu at (76.8, 115.1)
- added D2: LED_PWR, LED_SMD:LED_0603_1608Metric, F.Cu at (76.8, 113.1)
- added D3: LED_Cont., LED_SMD:LED_0603_1608Metric, F.Cu at (118.4, 100.3)
- added FB1: 180 @ 100 Mhz, Inductor_SMD:L_0603_1608Metric_Pad1.05x0.95mm_HandSolder, F.Cu at (94.4, 123.8)
- added J1: Debugger, Connector_PinHeader_2.54mm:PinHeader_2x05_P2.54mm_Vertical_SMD, F.Cu at (113.3, 80.0)
- added J2: Centroid, badger-connectors:CentroidPad-8-13mm, F.Cu at (100.0, 100.0)
- added J3: BATT, Connector_PinHeader_2.00mm:PinHeader_1x02_P2.00mm_Vertical, F.Cu at (66.4, 100.0)
- added J5: UART, Connector_PinHeader_2.54mm:PinHeader_1x03_P2.54mm_Vertical, F.Cu at (118.6, 97.1)
- added J7: GPIO, Connector_PinHeader_2.54mm:PinHeader_1x04_P2.54mm_Vertical, F.Cu at (85.4, 130.7)
- added L1: 4.7uH, Inductor_SMD:L_Vishay_IHLP-1616, F.Cu at (75.0, 97.5)
- added Q1: Q_NMOS_GDS, Package_TO_SOT_SMD:TO-263-3_TabPin2, F.Cu at (85.0, 79.5)
- added R1: 1.5k, Resistor_SMD:R_0402_1005Metric, F.Cu at (127.2, 92.1)
- added R10: 1.5k, Resistor_SMD:R_0402_1005Metric, F.Cu at (121.4, 100.3)
- added R2: 10k, Resistor_SMD:R_0402_1005Metric, F.Cu at (115.2, 92.1)
- added R3: 1.5k, Resistor_SMD:R_0402_1005Metric, F.Cu at (73.8, 115.1)
- added R4: 10k, Resistor_SMD:R_0402_1005Metric, F.Cu at (108.8, 86.7)
- added R5: 0R, Resistor_SMD:R_0402_1005Metric, F.Cu at (121.4, 80.6)
- added R6: 0R, Resistor_SMD:R_0402_1005Metric, F.Cu at (116.6, 112.4)
- added R7: 120R, Resistor_SMD:R_0402_1005Metric, F.Cu at (113.6, 108.8)
- added R8: 1.5k, Resistor_SMD:R_0402_1005Metric, F.Cu at (73.8, 113.1)
- added R9: 220R, Resistor_SMD:R_0402_1005Metric, F.Cu at (98.2, 115.7)
- added REF**: MountingHole_3.2mm_M3, MountingHole:MountingHole_3.2mm_M3, F.Cu at (100.2, 80.4)
- added SW1: BOOT, Button_Switch_SMD:SW_DIP_SPSTx01_Slide_6.7x4.1mm_W6.73mm_P2.54mm_LowProfile_JPin, F.Cu at (121.2, 92.1)
- added U1: STM32F103C8Tx, Package_QFP:LQFP-48_7x7mm_P0.5mm, F.Cu at (104.8, 118.0)
- added U2: SN65HVD230, Package_SO:SOIC-8_3.9x4.9mm_P1.27mm, F.Cu at (119.4, 108.8)
- added U3: AMS1117-3.3, Package_TO_SOT_SMD:SOT-223-3_TabPin2, F.Cu at (74.6, 105.7)
- added Y1: 8 Mhz 5032, Crystal:Crystal_SMD_5032-2Pin_5.0x3.2mm, F.Cu at (94.5, 118.0)
Routing:
- net GND: track 0.00 -> 64.8 mm, vias 0 -> 35
- net /MCU/UART_TX: track 0.00 -> 44.9 mm
- net Net-(R9-Pad2): track 0.00 -> 43.5 mm, vias 0 -> 2
- net /MCU/SWDIO: track 0.00 -> 43.2 mm, vias 0 -> 2
- net +3V3: track 0.00 -> 42.0 mm, vias 0 -> 17
- net /MCU/nRESET: track 0.00 -> 41.7 mm, vias 0 -> 2
- net /MCU/SWCLK: track 0.00 -> 39.9 mm, vias 0 -> 2
- net Net-(R2-Pad2): track 0.00 -> 36.9 mm, vias 0 -> 2
- net /MCU/UART_RX: track 0.00 -> 36.2 mm
- net /Ignition/BATT+: track 0.00 -> 36.1 mm, vias 0 -> 5
- net /MCU/SWO: track 0.00 -> 33.5 mm, vias 0 -> 2
- net /Ignition/CONT0: track 0.00 -> 28.7 mm, vias 0 -> 2
- net Net-(D1-Pad2): track 0.00 -> 26.4 mm, vias 0 -> 2
- net /MCU/CAN_RX: track 0.00 -> 25.6 mm
- net /Ignition/CONT_INDICATION: track 0.00 -> 25.0 mm, vias 0 -> 2
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- added copper zone on In2.Cu, net +3V3
- added copper zone on F.Cu, net /Ignition/BATT+
- added copper zone on In2.Cu, net /Ignition/BATT+
- added copper zone on B.Cu, net GND
- added copper zone on F.Cu, net GND
- added copper zone on In1.Cu, net GND
Other:
- board outline added: 70 x 70 mm
- copper layers 0 -> 4
- board text added: "."
- board text added: "0"
- board text added: "1"
- board text added: "2"
- board text added: "3"
- board text added: "3v3"
- board text added: "8"
- board text added: "BO"
- board text added: "BOOT"
- board text added: "Badger.Pike :Engine Control"
- board text added: "CONT."
- board text added: "CONTINUITY"
- board text added: "GPIO"
- board text added: "HeartBeat"
- board text added: "IGNITION"
- board text added: "MCU"
- board text added: "PWR"
- board text added: "Rev. 0"

Commit message: Update gitignore
Parts:
- added REF**: CP_Radial_D12.5mm_P5.00mm, Capacitor_THT:CP_Radial_D12.5mm_P5.00mm, F.Cu at (88.0, 76.3)
Other:
- board text added: "JLCJLCJLCJLC"

Commit message: Finish Engine Control Rev2
Parts:
- removed the REF** at (88.0, 76.3)
- added C13: 2000uF, Capacitor_THT:CP_Radial_D12.5mm_P5.00mm, F.Cu at (87.2, 85.2)
- added D4: LED_Charge, LED_SMD:LED_0603_1608Metric, F.Cu at (78.1, 92.9)
- added D5: LED_Discharge, LED_SMD:LED_0603_1608Metric, F.Cu at (102.3, 73.1)
- added Q2: Q_NMOS_GSD, Package_TO_SOT_SMD:SOT-23, F.Cu at (81.8, 90.1)
- added R11: 220R, Resistor_SMD:R_0402_1005Metric, F.Cu at (77.8, 91.1)
- added R12: 1.5k, Resistor_SMD:R_0402_1005Metric, F.Cu at (102.5, 74.7)
- added R13: 220R, Resistor_SMD:R_0402_1005Metric, F.Cu at (83.0, 93.4)
- added U4: CPC1135N, Package_SO:SOP-4_3.8x4.1mm_P2.54mm, F.Cu at (91.0, 72.9)
- Q1: value Q_NMOS_GDS -> Q_NMOS_GSD; footprint Package_TO_SOT_SMD:TO-263-3_TabPin2 -> Package_TO_SOT_SMD:SOT-23
- R9: value 220R -> 1.5k
- moved R9 28.5 mm to (81.2, 92.9)
- moved Q1 17.0 mm to (73.1, 91.7), turned to -90 degrees
Connections:
- J2 pad 2: Net-(Q1-Pad3) -> /Ignition/IGN+
- Q1 pad 1: Net-(R9-Pad2) -> Net-(D4-Pad2)
- Q1 pad 2: /Ignition/BATT+ -> Net-(C13-Pad1)
- Q1 pad 3: Net-(Q1-Pad3) -> /Ignition/BATT+
- R9 pad 1: /Ignition/IGN0 -> GND
- R9 pad 2: Net-(R9-Pad2) -> Net-(D4-Pad1)
- U1 pad 21: unconnected-(U1-Pad21) -> /MCU/SCL
- U1 pad 22: unconnected-(U1-Pad22) -> /MCU/SDA
- U1 pad 4: unconnected-(U1-Pad4) -> /Ignition/CHARGE
- U1 pad 46: unconnected-(U1-Pad46) -> /Ignition/nDISCHARGE
Routing:
- net /Ignition/nDISCHARGE: track 0.00 -> 55.8 mm, vias 0 -> 2
- net Net-(R9-Pad2): track 43.5 -> 0.00 mm, vias 2 -> 0
- net /Ignition/CHARGE: track 0.00 -> 39.7 mm, vias 0 -> 2
- net Net-(C13-Pad1): track 0.00 -> 32.0 mm
- net /Ignition/IGN0: track 1.95 -> 29.8 mm
- net /Ignition/BATT+: track 36.1 -> 11.6 mm, vias 5 -> 2
- net Net-(Q1-Pad3): track 18.4 -> 0.00 mm
- net Net-(D5-Pad2): track 0.00 -> 16.7 mm
- net /Ignition/IGN+: track 0.00 -> 15.6 mm
- net GND: track 64.8 -> 71.4 mm, vias 35 -> 45
- net Net-(D4-Pad2): track 0.00 -> 5.24 mm
- net Net-(Q2-Pad1): track 0.00 -> 2.85 mm
- net Net-(D4-Pad1): track 0.00 -> 1.75 mm
- net Net-(D5-Pad1): track 0.00 -> 1.66 mm
- added copper zone on B.Cu, net /Ignition/BATT+
- removed copper zone on F.Cu, net /Ignition/BATT+
- removed copper zone on In2.Cu, net /Ignition/BATT+
Other:
- board text added: "CHARGE"
- board text added: "DISCH."
- board text added: "Rev.2"
- board text removed: "Rev. 0"
